File: schematics/sensors_pcb/multiplexores.kicad_pcb (KiCad board)
At the start: 2 copper layers, 42 parts, among them J1 Conn_02x02_Odd_Even, J2 Screw_Terminal_01x02, M1 74LS165, M2 74LS165, M3 74LS165, M4 74LS165

Commit message: actualizo la placa por completo
Parts:
- moved R3 20.9 mm to (32.7, 50.7)
- moved R2 19.2 mm to (60.1, 48.6)
- moved R1 19.1 mm to (87.8, 48.6)
- moved R4 19.1 mm to (115.4, 48.6)
- moved Conn17 17.8 mm to (79.2, 64.0)
- moved Conn25 17.8 mm to (106.5, 64.0)
- moved Conn26 17.8 mm to (112.2, 64.0)
- moved Conn27 17.8 mm to (118.0, 64.0)
- moved Conn1 17.8 mm to (23.6, 63.9)
- moved Conn5 17.8 mm to (41.1, 21.4)
- moved M1 17.8 mm to (124.2, 38.8)
- moved Conn11 17.8 mm to (62.9, 64.0)
- moved Conn13 17.8 mm to (68.6, 21.4)
- moved Conn14 17.8 mm to (62.8, 21.4)
- moved Conn15 17.8 mm to (57.1, 21.4)
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- renumbered 1 to Conn1, 10 to Conn10, 11 to Conn11, 12 to Conn12, 13 to Conn13, 14 to Conn14, 15 to Conn15, 16 to Conn16, 17 to Conn17, 18 to Conn18, 19 to Conn19, 2 to Conn2, 20 to Conn20, 21 to Conn21, 22 to Conn22, 23 to Conn23, 24 to Conn24, 25 to Conn25, 26 to Conn26, 27 to Conn27, 28 to Conn28, 29 to Conn29, 3 to Conn3, 30 to Conn30, 31 to Conn31, 32 to Conn32, 5 to Conn5, 6 to Conn6, 8 to Conn8, 9 to Conn9, 4 to conn4, 7 to conn7
Connections:
- M1 pad 7: Net-(M1-Pad7) -> unconnected-(M1-Pad7)
- M2 pad 7: Net-(M2-Pad7) -> unconnected-(M2-Pad7)
- M3 pad 7: Net-(M3-Pad7) -> unconnected-(M3-Pad7)
- M4 pad 10: Net-(M4-Pad10) -> unconnected-(M4-Pad10)
- M4 pad 7: Net-(M4-Pad7) -> unconnected-(M4-Pad7)
Routing:
- net GND: track 339.0 -> 359.6 mm
- net /CEP(D15): track 123.2 -> 140.3 mm
- net /Vcc: track 395.2 -> 412.1 mm
- net /CP(D4): track 127.0 -> 143.2 mm
- net /DPA(D2): track 32.7 -> 42.9 mm
- net /LP(D5): track 108.9 -> 118.1 mm
- net /DS3B: track 2.89 -> 7.11 mm
- net /DS2A: track 21.3 -> 24.2 mm
- net /D12: track 14.3 -> 17.2 mm
- net /D29: track 14.4 -> 17.3 mm
- net /D1: track 14.5 -> 17.3 mm
- net /D21: track 14.5 -> 17.2 mm
- net /D13: track 14.4 -> 17.1 mm
- net /D16: track 14.4 -> 17.1 mm
- net /D20: track 14.4 -> 17.1 mm
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- added copper zone on B.Cu, net GND
Other:
- net class Default removed
