File: schematics/sensors_pcb/multiplexores.kicad_pcb (KiCad board)
At the start: 2 copper layers, 42 parts, among them J1 Conn_02x02_Odd_Even, J2 Screw_Terminal_01x02, M1 74LS165, M2 74LS165, M3 74LS165, M4 74LS165

Commit message: cvd
Parts:
- removed J1: Conn_02x02_Odd_Even, Connector_IDC:IDC-Header_2x03_P2.54mm_Vertical
- J2: value Screw_Terminal_01x02 -> Conn_02x03_Odd_Even; footprint TerminalBlock:TerminalBlock_bornier-2_P5.08mm -> Connector_IDC:IDC-Header_2x03_P2.54mm_Vertical
- moved J2 16.0 mm to (136.9, 32.8), turned to 0 degrees
Connections:
- J2 pad 1: GND -> /LP(D5)
- J2 pad 2: /Vcc -> /CP(D4)
Routing:
- net GND: track 359.6 -> 304.8 mm, vias 0 -> 2
- net /Vcc: track 412.1 -> 428.7 mm
- net /DPA(D2): track 42.9 -> 43.5 mm, vias 0 -> 3
Other:
- board text removed: "VCC GND"
