File: schematics/sensors_pcb/multiplexores.kicad_sch (KiCad schematic)
At the start: 42 parts

Commit message: cvd
Parts:
- removed J1: (no value), symbol Connector_Generic:Conn_02x02_Odd_Even
- removed J2: (no value), symbol Connector:Screw_Terminal_01x02
- added J2: Conn_02x03_Odd_Even, Connector_IDC:IDC-Header_2x03_P2.54mm_Vertical, symbol Connector_Generic:Conn_02x03_Odd_Even
- Conn1: value (none) -> 1; footprint (none) -> Connector_PinSocket_2.54mm:PinSocket_1x03_P2.54mm_Vertical
- Conn10: value (none) -> 10; footprint (none) -> Connector_PinSocket_2.54mm:PinSocket_1x03_P2.54mm_Vertical
- Conn11: value (none) -> 11; footprint (none) -> Connector_PinSocket_2.54mm:PinSocket_1x03_P2.54mm_Vertical
- Conn12: value (none) -> 12; footprint (none) -> Connector_PinSocket_2.54mm:PinSocket_1x03_P2.54mm_Vertical
- Conn13: value (none) -> 13; footprint (none) -> Connector_PinSocket_2.54mm:PinSocket_1x03_P2.54mm_Vertical
- Conn14: value (none) -> 14; footprint (none) -> Connector_PinSocket_2.54mm:PinSocket_1x03_P2.54mm_Vertical
- Conn15: value (none) -> 15; footprint (none) -> Connector_PinSocket_2.54mm:PinSocket_1x03_P2.54mm_Vertical
- Conn16: value (none) -> 16; footprint (none) -> Connector_PinSocket_2.54mm:PinSocket_1x03_P2.54mm_Vertical
- Conn17: value (none) -> 17; footprint (none) -> Connector_PinSocket_2.54mm:PinSocket_1x03_P2.54mm_Vertical
- Conn18: value (none) -> 18; footprint (none) -> Connector_PinSocket_2.54mm:PinSocket_1x03_P2.54mm_Vertical
- Conn19: value (none) -> 19; footprint (none) -> Connector_PinSocket_2.54mm:PinSocket_1x03_P2.54mm_Vertical
- Conn2: value (none) -> 2; footprint (none) -> Connector_PinSocket_2.54mm:PinSocket_1x03_P2.54mm_Vertical
- Conn20: value (none) -> 20; footprint (none) -> Connector_PinSocket_2.54mm:PinSocket_1x03_P2.54mm_Vertical
- Conn21: value (none) -> 21; footprint (none) -> Connector_PinSocket_2.54mm:PinSocket_1x03_P2.54mm_Vertical
- Conn22: value (none) -> 22; footprint (none) -> Connector_PinSocket_2.54mm:PinSocket_1x03_P2.54mm_Vertical
- Conn23: value (none) -> 23; footprint (none) -> Connector_PinSocket_2.54mm:PinSocket_1x03_P2.54mm_Vertical
- Conn24: value (none) -> 24; footprint (none) -> Connector_PinSocket_2.54mm:PinSocket_1x03_P2.54mm_Vertical
- Conn25: value (none) -> 25; footprint (none) -> Connector_PinSocket_2.54mm:PinSocket_1x03_P2.54mm_Vertical
- Conn26: value (none) -> 26; footprint (none) -> Connector_PinSocket_2.54mm:PinSocket_1x03_P2.54mm_Vertical
- Conn27: value (none) -> 27; footprint (none) -> Connector_PinSocket_2.54mm:PinSocket_1x03_P2.54mm_Vertical
- Conn28: value (none) -> 28; footprint (none) -> Connector_PinSocket_2.54mm:PinSocket_1x03_P2.54mm_Vertical
- Conn29: value (none) -> 29; footprint (none) -> Connector_PinSocket_2.54mm:PinSocket_1x03_P2.54mm_Vertical
- Conn3: value (none) -> 3; footprint (none) -> Connector_PinSocket_2.54mm:PinSocket_1x03_P2.54mm_Vertical
- Conn30: value (none) -> 30; footprint (none) -> Connector_PinSocket_2.54mm:PinSocket_1x03_P2.54mm_Vertical
- Conn31: value (none) -> 31; footprint (none) -> Connector_PinSocket_2.54mm:PinSocket_1x03_P2.54mm_Vertical
- Conn32: value (none) -> 32; footprint (none) -> Connector_PinSocket_2.54mm:PinSocket_1x03_P2.54mm_Vertical
- Conn5: value (none) -> 5; footprint (none) -> Connector_PinSocket_2.54mm:PinSocket_1x03_P2.54mm_Vertical
- Conn6: value (none) -> 6; footprint (none) -> Connector_PinSocket_2.54mm:PinSocket_1x03_P2.54mm_Vertical
- Conn8: value (none) -> 8; footprint (none) -> Connector_PinSocket_2.54mm:PinSocket_1x03_P2.54mm_Vertical
- Conn9: value (none) -> 9; footprint (none) -> Connector_PinSocket_2.54mm:PinSocket_1x03_P2.54mm_Vertical
- M1, M2, M3, M4: value (none) -> 74LS165; footprint (none) -> Package_DIP:DIP-16_W7.62mm_Socket_LongPads
- R1, R2, R3, R4: value (none) -> 15; footprint (none) -> extensores:extensor 15mm
- conn4: value (none) -> 4; footprint (none) -> Connector_PinSocket_2.54mm:PinSocket_1x03_P2.54mm_Vertical
- conn7: value (none) -> 7; footprint (none) -> Connector_PinSocket_2.54mm:PinSocket_1x03_P2.54mm_Vertical
Connections:
- net CEP(D15): now also J2.3 (Pin_3)
- net CP(D4): now also J2.2 (Pin_2)
- net DPA(D2): now also J2.4 (Pin_4)
- net GND: now also J2.5 (Pin_5)
- net LP(D5): now also J2.1 (Pin_1)
- net Vcc: now also J2.6 (Pin_6)
