File: schematics/Esp32_pcb/esp32.kicad_pcb (KiCad board)
At the start: 2 copper layers, 4 parts, among them J1 Conn_02x05_Odd_Even, J2 Conn_01x04_Female, J3 Screw_Terminal_01x02, U1 ESP32-Devkit-V1

Commit message: actualizo la placa por completo
Routing:
- net /Vcc: track 86.7 -> 94.3 mm
- net /SDA: track 14.9 -> 17.8 mm
- net GND: track 62.2 -> 61.6 mm
Other:
- net class Default removed

Commit message: cvd
Parts:
- J1: value Conn_02x05_Odd_Even -> Conn_02x03_Odd_Even; footprint Connector_IDC:IDC-Header_2x05_P2.54mm_Vertical -> Connector_IDC:IDC-Header_2x03_P2.54mm_Vertical
- J3: value Screw_Terminal_01x02 -> USB_B; footprint TerminalBlock:TerminalBlock_bornier-2_P5.08mm -> Connector_USB:USB_B_Lumberg_2411_02_Horizontal
- moved J1 10.4 mm to (87.4, 91.9), turned to 180 degrees
- moved J3 2.37 mm to (86.4, 73.3), turned to 90 degrees
Connections:
- J1 pad 1: Net-(J1-Pad1) -> /LP(D4)
- J1 pad 2: Net-(J1-Pad2) -> /CP(D5)
- J1 pad 3: Net-(J1-Pad3) -> /CEP(D15)
- J1 pad 4: /CEP(D15) -> /DP(D2)
- J1 pad 5: Net-(J1-Pad5) -> /Vcc
- J1 pad 6: /DP(D2) -> GND
- J3 pad 2: GND -> unconnected-(J3-Pad2)
- U1 pad 1: Net-(U1-Pad1) -> unconnected-(U1-Pad1)
- U1 pad 10: Net-(U1-Pad10) -> unconnected-(U1-Pad10)
- U1 pad 11: Net-(U1-Pad11) -> unconnected-(U1-Pad11)
- U1 pad 12: Net-(U1-Pad12) -> unconnected-(U1-Pad12)
- U1 pad 13: Net-(U1-Pad13) -> unconnected-(U1-Pad13)
- U1 pad 14: Net-(U1-Pad14) -> unconnected-(U1-Pad14)
- U1 pad 15: Net-(U1-Pad15) -> unconnected-(U1-Pad15)
- U1 pad 16: Net-(U1-Pad16) -> unconnected-(U1-Pad16)
- U1 pad 18: Net-(U1-Pad18) -> unconnected-(U1-Pad18)
- U1 pad 19: Net-(U1-Pad19) -> unconnected-(U1-Pad19)
- U1 pad 2: Net-(U1-Pad2) -> unconnected-(U1-Pad2)
- U1 pad 21: Net-(U1-Pad21) -> unconnected-(U1-Pad21)
- U1 pad 22: Net-(U1-Pad22) -> unconnected-(U1-Pad22)
- U1 pad 24: Net-(U1-Pad24) -> unconnected-(U1-Pad24)
- U1 pad 25: Net-(U1-Pad25) -> unconnected-(U1-Pad25)
- U1 pad 3: Net-(U1-Pad3) -> unconnected-(U1-Pad3)
- U1 pad 4: Net-(U1-Pad4) -> unconnected-(U1-Pad4)
- U1 pad 5: Net-(U1-Pad5) -> unconnected-(U1-Pad5)
- U1 pad 6: Net-(U1-Pad6) -> unconnected-(U1-Pad6)
- U1 pad 7: Net-(U1-Pad7) -> unconnected-(U1-Pad7)
- U1 pad 8: Net-(U1-Pad8) -> unconnected-(U1-Pad8)
- U1 pad 9: Net-(U1-Pad9) -> unconnected-(U1-Pad9)
Routing:
- net /DP(D2): track 11.6 -> 44.8 mm, vias 0 -> 2
- net GND: track 61.6 -> 71.5 mm
- net /Vcc: track 94.3 -> 103.8 mm, vias 0 -> 2
- net /CEP(D15): track 11.6 -> 14.8 mm
- net /CP(D5): track 19.1 -> 18.2 mm
