File: schematics/Esp32_pcb/esp32.kicad_sch (KiCad schematic)
At the start: 4 parts

Commit message: cvd
Parts:
- removed J1: (no value), symbol Connector_Generic:Conn_02x05_Odd_Even
- removed J3: (no value), symbol Connector:Screw_Terminal_01x02
- added J1: Conn_02x03_Odd_Even, Connector_IDC:IDC-Header_2x03_P2.54mm_Vertical, symbol Connector_Generic:Conn_02x03_Odd_Even
- added J3: USB_B, Connector_USB:USB_B_Lumberg_2411_02_Horizontal, symbol Connector:USB_B
- J2: value (none) -> Conn_01x04_Female; footprint (none) -> Connector_PinHeader_2.54mm:PinHeader_1x04_P2.54mm_Vertical
- U1: value (none) -> ESP32-Devkit-V1; footprint (none) -> DOIT_ESP32:DOIT_ESP32_Devkit
Connections:
- net CEP(D15): now also J1.3 (Pin_3)
- net CP(D5): now also J1.2 (Pin_2)
- net DP(D2): now also J1.4 (Pin_4)
- net GND: now also J1.6 (Pin_6), J3.4 (GND)
- net LP(D4): now also J1.1 (Pin_1)
- net Vcc: now also J1.5 (Pin_5), J3.1 (VBUS)
Changed lines of the file:
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@@
     (stroke (width 0) (type default) (color 0 0 0 0))
   )
-  (polyline (pts (xy 168.275 88.9) (xy 139.065 88.9))
+  (polyline (pts (xy 168.402 98.298) (xy 133.35 98.298))
     (stroke (width 0) (type default) (color 0 0 0 0))
   )
@@
     (stroke (width 0) (type default) (color 0 0 0 0))
   )
-  (polyline (pts (xy 139.065 50.8) (xy 168.275 50.8))
-    (stroke (width 0) (type default) (color 0 0 0 0))
-  )
-  (polyline (pts (xy 168.275 50.8) (xy 168.275 88.9))
-    (stroke (width 0) (type default) (color 0 0 0 0))
-  )
-  (polyline (pts (xy 139.065 88.9) (xy 139.065 50.8))
+  (polyline (pts (xy 133.223 50.8) (xy 168.275 50.8))
+    (stroke (width 0) (type default) (color 0 0 0 0))
+  )
+  (polyline (pts (xy 168.275 50.8) (xy 168.402 98.298))
+    (stroke (width 0) (type default) (color 0 0 0 0))
+  )
+  (polyline (pts (xy 133.35 98.298) (xy 133.223 50.8))
     (stroke (width 0) (type default) (color 0 0 0 0))
   )
@@
     (stroke (width 0) (type default) (color 0 0 0 0))
   )
-  (text "Conectores\n" (at 156.845 88.265 0)
+  (text "Conectores\n" (at 157.226 97.536 0)
     (effects (font (size 1.27 1.27)) (justify left bottom))
   )
@@
     (effects (font (size 1.27 1.27)) (justify left bottom))
   )
-  (label "DP(D2)" (at 159.385 78.74 0)
+  (label "DP(D2)" (at 157.734 73.914 0)
     (effects (font (size 1.27 1.27)) (justify left bottom))
   )
@@
     (effects (font (size 1.27 1.27)) (justify right bottom))
   )
-  (label "LP(D4)" (at 159.385 83.82 0)
-    (effects (font (size 1.27 1.27)) (justify left bottom))
-  )
-  (label "GND" (at 162.8648 58.8518 0)
-    (effects (font (size 1.27 1.27)) (justify left bottom))
-  )
-  (label "Vcc" (at 162.8648 61.3918 0)
-    (effects (font (size 1.27 1.27)) (justify left bottom))
+  (label "LP(D4)" (at 145.034 71.374 180)
+    (effects (font (size 1.27 1.27)) (justify right bottom))
   )
   (label "LP(D4)" (at 74.93 82.55 180)
@@
     (effects (font (size 1.27 1.27)) (justify right bottom))
   )
+  (label "GND" (at 157.734 76.454 0)
+    (effects (font (size 1.27 1.27)) (justify left bottom))
+  )
   (label "GND" (at 113.03 67.31 0)
     (effects (font (size 1.27 1.27)) (justify left bottom))
@@
     (effects (font (size 1.27 1.27)) (justify right bottom))
   )
-  (label "CEP(D15)" (at 159.385 76.2 0)
+  (label "Vcc" (at 145.034 76.454 180)
+    (effects (font (size 1.27 1.27)) (justify right bottom))
+  )
+  (label "CEP(D15)" (at 145.034 73.914 180)
+    (effects (font (size 1.27 1.27)) (justify right bottom))
+  )
+  (label "GND" (at 161.798 89.408 0)
     (effects (font (size 1.27 1.27)) (justify left bottom))
   )
@@
     (effects (font (size 1.27 1.27)) (justify right bottom))
   )
+  (label "Vcc" (at 146.558 81.788 180)
+    (effects (font (size 1.27 1.27)) (justify right bottom))
+  )
   (label "SDA" (at 113.03 74.93 0)
     (effects (font (size 1.27 1.27)) (justify left bottom))
@@
     (effects (font (size 1.27 1.27)) (justify left bottom))
   )
-  (label "CP(D5)" (at 146.685 83.82 180)
-    (effects (font (size 1.27 1.27)) (justify right bottom))
+  (label "CP(D5)" (at 157.734 71.374 0)
+    (effects (font (size 1.27 1.27)) (justify left bottom))
   )
   (global_label "GND" (shape input) (at 119.38 67.31 0) (fields_autoplaced)
@@
       (effects (font (size 1.524 1.524)) hide)
     )
-    (property "Value" "" (id 1) (at 93.98 57.277 0)
+    (property "Value" "ESP32-Devkit-V1" (id 1) (at 93.98 57.277 0)
       (effects (font (size 2.0066 2.0066)))
     )
-    (property "Footprint" "" (id 2) (at 80.01 59.69 0)
+    (property "Footprint" "DOIT_ESP32:DOIT_ESP32_Devkit" (id 2) (at 80.01 59.69 0)
       (effects (font (size 1.524 1.524)) hide)
     )
@@
       (effects (font (size 1.27 1.27)) (justify left))
     )
-    (property "Value" "" (id 1) (at 150.876 61.2648 0)
+    (property "Value" "Conn_01x04_Female" (id 1) (at 150.876 61.2648 0)
       (effects (font (size 1.27 1.27)) (justify left) hide)
     )
-    (property "Footprint" "" (id 2) (at 150.1648 58.3438 0)
+    (property "Footprint" "Connector_PinHeader_2.54mm:PinHeader_1x04_P2.54mm_Vertical" (id 2) (at 150.1648 58.3438 0)
       (effects (font (size 1.27 1.27)) hide)
     )
@@
     (pin "4")
   )
-  (symbol (lib_id "Connector_Generic:Conn_02x05_Odd_Even") (at 151.765 78.74 0) (unit 1)
-    (in_bom yes) (on_board yes)
-    (property "Reference" "J1" (id 0) (at 153.035 68.1482 0))
-    (property "Value" "" (id 1) (at 153.035 70.4596 0))
-    (property "Footprint" "" (id 2) (at 151.765 78.74 0)
-      (effects (font (size 1.27 1.27)) hide)
-    )
-    (property "Datasheet" "~" (id 3) (at 151.765 78.74 0)
-      (effects (font (size 1.27 1.27)) hide)
-    )
-    (pin "1")
-    (pin "10")
+  (symbol (lib_id "Connector:USB_B") (at 151.638 89.408 90) (unit 1)
+    (in_bom yes) (on_board yes) (fields_autoplaced)
+    (property "Reference" "J3" (id 0) (at 142.494 88.1379 90)
+      (effects (font (size 1.27 1.27)) (justify left))
+    )
+    (property "Value" "USB_B" (id 1) (at 142.494 90.6779 90)
+      (effects (font (size 1.27 1.27)) (justify left))
+    )
+    (property "Footprint" "Connector_USB:USB_B_Lumberg_2411_02_Horizontal" (id 2) (at 152.908 85.598 0)
+      (effects (font (size 1.27 1.27)) hide)
+    )
+    (property "Datasheet" " ~" (id 3) (at 152.908 85.598 0)
+      (effects (font (size 1.27 1.27)) hide)
+    )
+    (pin "1")
+    (pin "2")
+    (pin "3")
+    (pin "4")
+    (pin "5")
+  )
+  (symbol (lib_id "Connector_Generic:Conn_02x03_Odd_Even") (at 150.114 73.914 0) (unit 1)
+    (in_bom yes) (on_board yes) (fields_autoplaced)
+    (property "Reference" "J1" (id 0) (at 151.384 64.262 0))
+    (property "Value" "Conn_02x03_Odd_Even" (id 1) (at 151.384 66.802 0))
+    (property "Footprint" "Connector_IDC:IDC-Header_2x03_P2.54mm_Vertical" (id 2) (at 150.114 73.914 0)
+      (effects (font (size 1.27 1.27)) hide)
+    )
+    (property "Datasheet" "~" (id 3) (at 150.114 73.914 0)
+      (effects (font (size 1.27 1.27)) hide)
+    )
+    (pin "1")
     (pin "2")
     (pin "3")
@@
     (pin "5")
     (pin "6")
-    (pin "7")
-    (pin "8")
-    (pin "9")
-  )
-  (symbol (lib_id "Connector:Screw_Terminal_01x02") (at 157.7848 61.3918 180) (unit 1)
-    (in_bom yes) (on_board yes)
-    (property "Reference" "J3" (id 0) (at 159.8676 55.4736 0))
-    (property "Value" "" (id 1) (at 155.7528 58.8772 0)
-      (effects (font (size 1.27 1.27)) (justify left) hide)
-    )
-    (property "Footprint" "" (id 2) (at 157.7848 61.3918 0)
-      (effects (font (size 1.27 1.27)) hide)
-    )
-    (property "Datasheet" "~" (id 3) (at 157.7848 61.3918 0)
-      (effects (font (size 1.27 1.27)) hide)
-    )
-    (pin "1")
-    (pin "2")
   )
   (sheet_instances
@@
   )
   (symbol_instances
-    (path "/00000000-0000-0000-0000-000060fb67cb"
-      (reference "J1") (unit 1) (value "Conn_02x05_Odd_Even") (footprint "Connector_IDC:IDC-Header_2x05_P2.54mm_Vertical")
+    (path "/b22cddd5-ec6d-4290-9c9a-471c435e7a95"
+      (reference "J1") (unit 1) (value "Conn_02x03_Odd_Even") (footprint "Connector_IDC:IDC-Header_2x03_P2.54mm_Vertical")
     )
     (path "/00000000-0000-0000-0000-000060fb18e8"
       (reference "J2") (unit 1) (value "Conn_01x04_Female") (footprint "Connector_PinHeader_2.54mm:PinHeader_1x04_P2.54mm_Vertical")
     )
-    (path "/00000000-0000-0000-0000-00006110b675"
-      (reference "J3") (unit 1) (value "Screw_Terminal_01x02") (footprint "TerminalBlock:TerminalBlock_bornier-2_P5.08mm")
+    (path "/7e422374-3dc9-4db5-b492-3950f5c41afa"
+      (reference "J3") (unit 1) (value "USB_B") (footprint "Connector_USB:USB_B_Lumberg_2411_02_Horizontal")
     )
     (path "/00000000-0000-0000-0000-000060fafda6"
